Commit message: update link urdfs for common plan generation

File: urdf/pole_2_links_7DOF/pole_2_links.urdf (robot description, URDF)
Before this commit: robot pole, 17 links, 16 joints
Links:
- removed link tool1
- added link pole_holder_link_34
- added link pole_holder_link_5
- added link tool00
Joints:
- removed joint joint_link_right_1_root_back_to_tool1
- removed joint spherical_to_tool0
- removed joint tool0_to_link_left_1_root
- added joint joint_link_right_1_root_back_to_tool0: type fixed, parent link_right_1_root_back, child tool0, origin xyz=0 0 0 rpy=0 0 0
- added joint pole_holder_fixed_joint_34: type fixed, parent link_left_1_root_back, child pole_holder_link_34, origin xyz=0 0 1.21539 rpy=0 0 0
- added joint pole_holder_fixed_joint_5: type fixed, parent link_right_1_root_back, child pole_holder_link_5, origin xyz=0 0 -1.2153899999999997 rpy=0 0 0
- added joint spherical_to_tool00: type fixed, parent spherical_roll_link, child tool00, origin xyz=0 0 0 rpy=0 0 0
- added joint tool00_to_link_left_1_root: type fixed, parent tool00, child link_left_1_root, origin xyz=0 0 0 rpy=0 0 0

File: urdf/pole_2_links_9DOF/pole_2_links.urdf (robot description, URDF)
Before this commit: robot pole, 19 links, 18 joints
Links:
- removed link tool1
- added link pole_holder_link_34
- added link pole_holder_link_5
- added link tool00
Joints:
- removed joint joint_link_right_1_root_back_to_tool1
- removed joint spherical_to_tool0
- removed joint tool0_to_link_left_1_root
- added joint joint_link_right_1_root_back_to_tool0: type fixed, parent link_right_1_root_back, child tool0, origin xyz=0 0 0 rpy=0 0 0
- added joint pole_holder_fixed_joint_34: type fixed, parent link_left_1_root_back, child pole_holder_link_34, origin xyz=0 0 1.21539 rpy=0 0 0
- added joint pole_holder_fixed_joint_5: type fixed, parent link_right_1_root_back, child pole_holder_link_5, origin xyz=0 0 -1.2153899999999997 rpy=0 0 0
- added joint spherical_to_tool00: type fixed, parent spherical_roll_link, child tool00, origin xyz=0 0 0 rpy=0 0 0
- added joint tool00_to_link_left_1_root: type fixed, parent tool00, child link_left_1_root, origin xyz=0 0 0 rpy=0 0 0
