Commit message: Update dlo kinematic model with 3 rev joints instead of 2

File: src/dlo_urdf_creator/dlo_urdf_equal_segment_length.urdf (robot description, URDF)
Before this commit: robot pole, 50 links, 49 joints
Links:
- removed link pole_link_35
- removed link pole_link_36
- removed link pole_link_37
- removed link pole_link_38
- removed link pole_link_39
- removed link pole_link_40
- removed link pole_link_41
- removed link pole_link_42
- removed link pole_link_43
- removed link pole_link_44
- link pole_link_11: geometry 
- link pole_link_12: geometry collision cylinder length=0.098 radius=0.01; visual cylinder length=0.098 radius=0.01
- link pole_link_13: geometry 
- link pole_link_15: geometry collision cylinder length=0.098 radius=0.01; visual cylinder length=0.098 radius=0.01
- link pole_link_17: geometry 
- link pole_link_18: geometry collision cylinder length=0.098 radius=0.01; visual cylinder length=0.098 radius=0.01
- link pole_link_19: geometry 
- link pole_link_21: geometry collision cylinder length=0.098 radius=0.01; visual cylinder length=0.098 radius=0.01
- link pole_link_23: geometry 
- link pole_link_24: geometry collision cylinder length=0.098 radius=0.01; visual cylinder length=0.098 radius=0.01
- link pole_link_25: geometry 
- link pole_link_27: geometry collision cylinder length=0.098 radius=0.01; visual cylinder length=0.098 radius=0.01
- link pole_link_29: geometry 
- link pole_link_30: geometry collision cylinder length=0.098 radius=0.01; visual cylinder length=0.098 radius=0.01
- link pole_link_31: geometry 
- link pole_link_33: geometry collision cylinder length=0.098 radius=0.01; visual cylinder length=0.098 radius=0.01
- link pole_link_5: geometry 
- link pole_link_6: geometry collision cylinder length=0.098 radius=0.01; visual cylinder length=0.098 radius=0.01
- link pole_link_7: geometry 
- link pole_link_9: geometry collision cylinder length=0.098 radius=0.01; visual cylinder length=0.098 radius=0.01
Joints:
- removed joint pole_rev_joint_34
- removed joint pole_rev_joint_35
- removed joint pole_rev_joint_36
- removed joint pole_rev_joint_37
- removed joint pole_rev_joint_38
- removed joint pole_rev_joint_39
- removed joint pole_rev_joint_40
- removed joint pole_rev_joint_41
- removed joint pole_rev_joint_42
- removed joint pole_rev_joint_43
- joint pole_center_joint: origin xyz=0 0 0.049999999999999975 rpy=0 0 0 -> xyz=0 0 0.09999999999999998 rpy=0 0 0; parent pole_link_23 -> pole_link_18
- joint pole_end_joint: child pole_link_44 -> pole_link_34; origin xyz=0 0 0.05 rpy=0 0 0 -> xyz=0 0 0.1 rpy=0 0 0; parent pole_link_43 -> pole_link_33
- joint pole_holding_joint_1: origin xyz=0 0 0.012499999999999997 rpy=0 0 0 -> xyz=0 0 0.0625 rpy=0 0 0; parent pole_link_39 -> pole_link_30
- joint pole_rev_joint_10: origin xyz=0 0 0.05 -> xyz=0 0 0.1
- joint pole_rev_joint_12: axis 1 0 0 -> 0 0 1; limit lower=-1.5707963267948966 upper=1.5707963267948966 effort=100 velocity=1.0 -> lower=-0.17453292519943295 upper=0.17453292519943295 effort=100 velocity=1.0; origin xyz=0 0 0.05 -> xyz=0 0 0
- joint pole_rev_joint_13: axis 0 1 0 -> 1 0 0; limit lower=-3.141592653589793 upper=3.141592653589793 effort=100 velocity=1.0 -> lower=-1.5707963267948966 upper=1.5707963267948966 effort=100 velocity=1.0; origin xyz=0 0 0 -> xyz=0 0 0.1
- joint pole_rev_joint_14: axis 1 0 0 -> 0 1 0; limit lower=-1.5707963267948966 upper=1.5707963267948966 effort=100 velocity=1.0 -> lower=-3.141592653589793 upper=3.141592653589793 effort=100 velocity=1.0; origin xyz=0 0 0.05 -> xyz=0 0 0
- joint pole_rev_joint_15: axis 0 1 0 -> 0 0 1; limit lower=-3.141592653589793 upper=3.141592653589793 effort=100 velocity=1.0 -> lower=-0.17453292519943295 upper=0.17453292519943295 effort=100 velocity=1.0
- joint pole_rev_joint_16: origin xyz=0 0 0.05 -> xyz=0 0 0.1
- joint pole_rev_joint_18: axis 1 0 0 -> 0 0 1; limit lower=-1.5707963267948966 upper=1.5707963267948966 effort=100 velocity=1.0 -> lower=-0.17453292519943295 upper=0.17453292519943295 effort=100 velocity=1.0; origin xyz=0 0 0.05 -> xyz=0 0 0
- joint pole_rev_joint_19: axis 0 1 0 -> 1 0 0; limit lower=-3.141592653589793 upper=3.141592653589793 effort=100 velocity=1.0 -> lower=-1.5707963267948966 upper=1.5707963267948966 effort=100 velocity=1.0; origin xyz=0 0 0 -> xyz=0 0 0.1
- joint pole_rev_joint_20: axis 1 0 0 -> 0 1 0; limit lower=-1.5707963267948966 upper=1.5707963267948966 effort=100 velocity=1.0 -> lower=-3.141592653589793 upper=3.141592653589793 effort=100 velocity=1.0; origin xyz=0 0 0.05 -> xyz=0 0 0
- joint pole_rev_joint_21: axis 0 1 0 -> 0 0 1; limit lower=-3.141592653589793 upper=3.141592653589793 effort=100 velocity=1.0 -> lower=-0.17453292519943295 upper=0.17453292519943295 effort=100 velocity=1.0
- joint pole_rev_joint_22: origin xyz=0 0 0.05 -> xyz=0 0 0.1
- joint pole_rev_joint_24: axis 1 0 0 -> 0 0 1; limit lower=-1.5707963267948966 upper=1.5707963267948966 effort=100 velocity=1.0 -> lower=-0.17453292519943295 upper=0.17453292519943295 effort=100 velocity=1.0; origin xyz=0 0 0.05 -> xyz=0 0 0
- joint pole_rev_joint_25: axis 0 1 0 -> 1 0 0; limit lower=-3.141592653589793 upper=3.141592653589793 effort=100 velocity=1.0 -> lower=-1.5707963267948966 upper=1.5707963267948966 effort=100 velocity=1.0; origin xyz=0 0 0 -> xyz=0 0 0.1
- joint pole_rev_joint_26: axis 1 0 0 -> 0 1 0; limit lower=-1.5707963267948966 upper=1.5707963267948966 effort=100 velocity=1.0 -> lower=-3.141592653589793 upper=3.141592653589793 effort=100 velocity=1.0; origin xyz=0 0 0.05 -> xyz=0 0 0
- joint pole_rev_joint_27: axis 0 1 0 -> 0 0 1; limit lower=-3.141592653589793 upper=3.141592653589793 effort=100 velocity=1.0 -> lower=-0.17453292519943295 upper=0.17453292519943295 effort=100 velocity=1.0
- joint pole_rev_joint_28: origin xyz=0 0 0.05 -> xyz=0 0 0.1
- joint pole_rev_joint_30: axis 1 0 0 -> 0 0 1; limit lower=-1.5707963267948966 upper=1.5707963267948966 effort=100 velocity=1.0 -> lower=-0.17453292519943295 upper=0.17453292519943295 effort=100 velocity=1.0; origin xyz=0 0 0.05 -> xyz=0 0 0
- joint pole_rev_joint_31: axis 0 1 0 -> 1 0 0; limit lower=-3.141592653589793 upper=3.141592653589793 effort=100 velocity=1.0 -> lower=-1.5707963267948966 upper=1.5707963267948966 effort=100 velocity=1.0; origin xyz=0 0 0 -> xyz=0 0 0.1
- joint pole_rev_joint_32: axis 1 0 0 -> 0 1 0; limit lower=-1.5707963267948966 upper=1.5707963267948966 effort=100 velocity=1.0 -> lower=-3.141592653589793 upper=3.141592653589793 effort=100 velocity=1.0; origin xyz=0 0 0.05 -> xyz=0 0 0
- joint pole_rev_joint_33: axis 0 1 0 -> 0 0 1; limit lower=-3.141592653589793 upper=3.141592653589793 effort=100 velocity=1.0 -> lower=-0.17453292519943295 upper=0.17453292519943295 effort=100 velocity=1.0
- joint pole_rev_joint_6: axis 1 0 0 -> 0 0 1; limit lower=-1.5707963267948966 upper=1.5707963267948966 effort=100 velocity=1.0 -> lower=-3.141592653589793 upper=3.141592653589793 effort=100 velocity=1.0; origin xyz=0 0 0.05 -> xyz=0 0 0
- joint pole_rev_joint_7: axis 0 1 0 -> 1 0 0; limit lower=-3.141592653589793 upper=3.141592653589793 effort=100 velocity=1.0 -> lower=-1.5707963267948966 upper=1.5707963267948966 effort=100 velocity=1.0; origin xyz=0 0 0 -> xyz=0 0 0.1
- joint pole_rev_joint_8: axis 1 0 0 -> 0 1 0; limit lower=-1.5707963267948966 upper=1.5707963267948966 effort=100 velocity=1.0 -> lower=-3.141592653589793 upper=3.141592653589793 effort=100 velocity=1.0; origin xyz=0 0 0.05 -> xyz=0 0 0
- joint pole_rev_joint_9: axis 0 1 0 -> 0 0 1; limit lower=-3.141592653589793 upper=3.141592653589793 effort=100 velocity=1.0 -> lower=-0.17453292519943295 upper=0.17453292519943295 effort=100 velocity=1.0
- joint pole_tcp_joint: parent pole_link_44 -> pole_link_34
